File: piscine-electronique/project/piscine-electronique.kicad_pcb (KiCad board)
At the start: 2 copper layers, 17 parts, among them J3 FTDI, SW1 SW_Push, U1 ATmega328P-A, Y1 16MHz

Commit message: v final
Parts:
- moved J3 51.5 mm to (130.2, 107.1), turned to -90 degrees
- moved J1 48.2 mm to (140.7, 93.3)
- moved Y1 40.8 mm to (136.2, 94.2)
- moved C4 38.0 mm to (124.6, 92.6)
- moved SW1 36.6 mm to (124.5, 95.1)
- moved R3 36.4 mm to (124.4, 98.0)
- moved C1 33.2 mm to (136.0, 91.4), turned to 180 degrees
- moved C2 32.4 mm to (136.2, 97.0)
- moved C7 25.9 mm to (123.5, 102.3), turned to 180 degrees
- moved D1 24.6 mm to (125.4, 78.9), turned to -90 degrees
- moved J2 22.8 mm to (119.8, 93.2), turned to 180 degrees
- moved U1 22.1 mm to (129.9, 86.6), turned to 135 degrees
- moved C6 21.9 mm to (123.4, 100.7), turned to 180 degrees
- moved R1 17.7 mm to (127.3, 78.9), turned to -90 degrees
- moved R2 15.1 mm to (128.7, 104.1), turned to 180 degrees
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Routing:
- net DTR: track 4.53 -> 56.0 mm
- net GND: track 0.00 -> 41.2 mm
- net RXI: track 0.00 -> 39.0 mm
- net TXO: track 0.00 -> 30.5 mm
- net SCK: track 0.00 -> 21.8 mm
- net D10: track 0.00 -> 20.5 mm
- net MISO: track 0.00 -> 20.3 mm
- net MOSI: track 0.00 -> 20.1 mm
- net D4: track 0.00 -> 18.2 mm
- net D2: track 0.00 -> 16.4 mm
- net VCC: track 0.00 -> 16.4 mm
- net D3: track 0.00 -> 16.4 mm
- net A3: track 0.00 -> 11.1 mm
- net Net-(U1-XTAL1/PB6): track 0.00 -> 10.4 mm
- net D9: track 0.00 -> 9.81 mm
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Other:
- board outline added: 26.7 x 36.4 mm
- board text added: "ADAM"
